File: board/schematic/relay_shield.sch (KiCad schematic (older format))
At the start: 0 parts

Commit message: Added Spark Core library/component.
Parts:
- added U?: SPARK_CORE, ~, symbol SPARK_CORE
Connections:
- net labels added: +3.3V, CS, GND, RS, SS
- wire segments 0 -> 9
Other:
- note added: "RS: Read State of the relay.\nSS: Set State of the relay.\nCS: Current Sense."
Changed lines of the file:
@@
 LIBS:contrib
 LIBS:valves
+LIBS:spark_core
 LIBS:relay_shield-cache
 EELAYER 27 0
@@
 Comment4 ""
 $EndDescr
+$Comp
+L SPARK_CORE U?
+U 1 1 5209DC68
+P 7800 4850
+F 0 "U?" H 7800 4900 60  0000 C CNN
+F 1 "SPARK_CORE" H 7800 4100 60  0000 C CNN
+F 2 "~" H 8300 5050 60  0000 C CNN
+F 3 "~" H 8300 5050 60  0000 C CNN
+	1    7800 4850
+	1    0    0    -1
+$EndComp
+$Comp
+L +3.3V #PWR?
+U 1 1 5209DCD5
+P 8700 4200
+F 0 "#PWR?" H 8700 4160 30  0001 C CNN
+F 1 "+3.3V" H 8700 4310 30  0000 C CNN
+F 2 "" H 8700 4200 60  0000 C CNN
+F 3 "" H 8700 4200 60  0000 C CNN
+	1    8700 4200
+	1    0    0    -1
+$EndComp
+$Comp
+L GND #PWR?
+U 1 1 5209DCE7
+P 8700 4650
+F 0 "#PWR?" H 8700 4650 30  0001 C CNN
+F 1 "GND" H 8700 4580 30  0001 C CNN
+F 2 "" H 8700 4650 60  0000 C CNN
+F 3 "" H 8700 4650 60  0000 C CNN
+	1    8700 4650
+	1    0    0    -1
+$EndComp
+$Comp
+L GND #PWR?
+U 1 1 5209DD15
+P 6900 4450
+F 0 "#PWR?" H 6900 4450 30  0001 C CNN
+F 1 "GND" H 6900 4380 30  0001 C CNN
+F 2 "" H 6900 4450 60  0000 C CNN
+F 3 "" H 6900 4450 60  0000 C CNN
+	1    6900 4450
+	1    0    0    -1
+$EndComp
+Wire Wire Line
+	8700 4650 8700 4600
+Wire Wire Line
+	8700 4600 8450 4600
+Wire Wire Line
+	8450 4300 8700 4300
+Wire Wire Line
+	8700 4300 8700 4200
+Wire Wire Line
+	7150 4400 6900 4400
+Wire Wire Line
+	6900 4400 6900 4450
+Wire Wire Line
+	8450 5400 8700 5400
+Wire Wire Line
+	7150 5400 6900 5400
+Wire Wire Line
+	8450 5300 8700 5300
+Text Label 8600 5300 0    60   ~ 0
+RS
+Text Label 8600 5400 0    60   ~ 0
+SS
+Text Label 6900 5400 0    60   ~ 0
+CS
+Text Notes 8300 5700 0    60   ~ 0
+RS: Read State of the relay.\nSS: Set State of the relay.\nCS: Current Sense.
 $EndSCHEMATC

Commit message: Optoisolator version. Not sure if to follow that path.
Parts:
- added C?: 10uF, ~, symbol CP1
- added D?: LED, ~, symbol LED
- added D?: 1N4148, ~, symbol DIODE
- added P?: CT, symbol CONN_2
- added Q?: 2N3904, ~, symbol NPN
- added R? (x2): 1K, ~, symbol R
- added R? (x4): 10K, ~, symbol R
- added R?: 220, ~, symbol R
- added R?: 18 - 1%, ~, symbol R
- added SW?: SPST, ~, symbol SPST
- added U?: Optoisolator, ~, symbol PHDARL
Connections:
- net labels added: +5V
- wire segments 9 -> 35
Other:
- note added: "->\n"
- note added: "<-"
- note added: "MCP1825S 500 mA LDO\n"
