File: board/kicad/relay_shield.kicad_pcb (KiCad board)
At the start: 2 copper layers, 100.3 x 38.1 mm, 22 parts, among them P1 CT, P2 Z1, P3 Z2, P4 AC, P5 MH1, P6 MH2, P7 MH3, P8 MH4, P9 PWR, Q1 2N3904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

Commit message: Finished to route the board.
Parts:
- turned P9 to 0 degrees
Routing:
- net /CS: track 0.00 -> 115.5 mm
- net +5V: track 0.00 -> 84.8 mm
- net N-000003: track 0.00 -> 73.8 mm
- net GND: track 0.00 -> 59.9 mm
- net +3.3V: track 0.00 -> 32.4 mm
- net N-000001: track 0.00 -> 30.6 mm
- net /RS: track 0.00 -> 25.6 mm
- net N-0000027: track 0.00 -> 22.9 mm
- net N-0000035: track 0.00 -> 20.1 mm
- net N-0000033: track 0.00 -> 9.20 mm
- net N-0000032: track 0.00 -> 7.62 mm
- added copper zone on B.Cu, net GND
Other:
- net class AC power added: clearance 2.54, trace_width 5.08, via_dia 0.889, via_drill 0.635
