File: board/kicad/relay_shield.kicad_pcb (KiCad board)
At the start: 2 copper layers, 100.3 x 38.1 mm, 22 parts, among them P1 CT, P2 Z1, P3 Z2, P4 AC, P5 MH1, P6 MH2, P7 MH3, P8 MH4, P9 PWR, Q1 2N3904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

Commit message: Finished the Silkscreen.
Parts:
- added G***: high_voltage_logo, high_voltage_logo, F.Cu at (102.6, 92.7)
- added G*** (x2): oshw_logo, oshw_logo, F.Cu at (133.1, 77.5)
- moved P1 42.5 mm to (102.6, 109.2)
- moved P6 42.5 mm to (187.7, 77.5)
- moved P7 42.5 mm to (187.7, 108.0)
- moved Q1 42.5 mm to (145.8, 101.6)
- moved R1 42.5 mm to (156.0, 88.9)
- moved R6 42.5 mm to (145.8, 88.9)
- moved P2 42.5 mm to (95.0, 87.6)
- moved P3 42.5 mm to (95.0, 97.8)
- moved P4 42.5 mm to (102.6, 92.7)
- moved P5 42.5 mm to (95.0, 77.5)
- moved P8 42.5 mm to (95.0, 108.0)
- moved P9 42.5 mm to (153.4, 109.2)
- moved R3 42.5 mm to (144.5, 109.2)
- moved RE1 42.5 mm to (124.2, 91.4)
- moved C1 42.5 mm to (153.4, 100.3)
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Other:
- board text added: "Advanced Relay Shield"
- board text added: "By Carlos Jenkins"
- board text added: "goo.gl/66vFVi"
- board text added: "v0.1"
