File: board/kicad/relay_shield.kicad_pcb (KiCad board)
At the start: 2 copper layers, 100.3 x 38.1 mm, 25 parts, among them P1 CT, P2 Z1, P3 Z2, P4 AC, P5 MH1, P6 MH2, P7 MH3, P8 MH4, P9 PWR, Q1 2N3904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

Commit message: Added extra pads to allow connection to unused pins. Also fixed stand-offs size.
Parts:
- removed G***: oshw_logo, oshw_logo
- added OSHW: oshw_logo, oshw_logo, F.Cu at (133.1, 77.5)
- U1: footprint SPARK_CORE -> SPARK_CORE_EX
- renumbered G*** to OSHW_M, G*** to WARN
Routing:
- net GND: track 59.9 -> 80.0 mm
- net /RS: track 25.6 -> 30.7 mm
- net +5V: track 84.8 -> 87.3 mm
- net +3.3V: track 32.4 -> 34.9 mm
- net /CS: track 115.5 -> 117.6 mm

Commit message: Rolled out v1.0.
Routing:
- net /CS: track 117.6 -> 120.1 mm
Other:
- board text added: "v1.0"
- board text removed: "v0.1"
